Commit message: prelim first evolution algorithm

File: urdf/rupert.xacro (robot description, xacro)
@@ -7,23 +7,28 @@
   <xacro:property name="width" value="0.1" /> <!-- Square dimensions (widthxwidth) of beams -->
   <!--Body -->
+  <xacro:property name="mass_body" value="1" />
   <xacro:property name="body_width" value="0.81" /> <!-- width of body -->
   <xacro:property name="body_length" value="1.13" /> <!-- length of body -->
   <xacro:property name="body_height" value="0.25" /> <!-- height of body -->
   <!--block -->
-  <xacro:property name="block_width" value="0.22" /> <!-- width of body -->
-  <xacro:property name="block_length" value="0.17" /> <!-- length of body -->
-  <xacro:property name="block_height" value="0.25" /> <!-- height of body -->
+  <xacro:property name="mass_block" value="1" />
+  <xacro:property name="block_width" value="0.22" /> <!-- width of block -->
+  <xacro:property name="block_length" value="0.17" /> <!-- length of  block -->
+  <xacro:property name="block_height" value="0.25" /> <!-- height of block -->
   <!--Hip -->
-  <xacro:property name="hip_width" value="0.4" /> <!-- width of body -->
-  <xacro:property name="hip_length" value="0.4" /> <!-- length of body -->
-  <xacro:property name="hip_height" value="0.4" /> <!-- height of body -->
+  <xacro:property name="mass_hip" value="1" />
+  <xacro:property name="hip_width" value="0.4" /> <!-- width of hip -->
+  <xacro:property name="hip_length" value="0.4" /> <!-- length of hip -->
+  <xacro:property name="hip_height" value="0.4" /> <!-- height of hip -->
   <!--leg -->
-  <xacro:property name="leg_width" value="0.25" /> <!-- width of body -->
-  <xacro:property name="leg_length" value="0.15" /> <!-- length of body -->
-  <xacro:property name="leg_height" value="0.45" /> <!-- height of body -->
+  <xacro:property name="mass_leg" value="1" />
+  <xacro:property name="leg_width" value="0.25" /> <!-- width of leg -->
+  <xacro:property name="leg_length" value="0.15" /> <!-- length of leg -->
+  <xacro:property name="leg_height" value="0.45" /> <!-- height of leg -->
     <!--foot -->
-  <xacro:property name="foot_width" value="0.01" /> <!-- width of body -->
-  <xacro:property name="foot_length" value="0.01" /> <!-- length of body -->
-  <xacro:property name="foot_height" value="0.75" /> <!-- height of body -->
+  <xacro:property name="mass_foot" value="1" />
+  <xacro:property name="foot_width" value="0.01" /> <!-- width of foot -->
+  <xacro:property name="foot_length" value="0.01" /> <!-- length of foot -->
+  <xacro:property name="foot_height" value="0.75" /> <!-- height of foot -->
   <xacro:property name="height1" value="0.0001" /> <!-- Link 1 -->
   <xacro:property name="height2" value="0.0005" /> <!-- Link 2 -->
@@ -57,9 +62,9 @@
     <inertial>
       <origin xyz="0 0 0" rpy="0 0 0"/>
-      <mass value="${mass}"/>
-      <inertia
-    ixx="${mass / 12.0*(body_length*body_length + body_height*body_height)}" ixy="0.0" ixz="0.0"
-    iyy="${mass / 12.0 * (body_height*body_height + body_width*body_width)}" iyz="0.0"
-    izz="${mass / 12.0 * (body_width*body_width + body_length*body_length)}"/>
+      <mass value="${mass_body}"/>
+      <inertia
+    ixx="${mass_body / 12.0*(body_length*body_length + body_height*body_height)}" ixy="0.0" ixz="0.0"
+    iyy="${mass_body / 12.0 * (body_height*body_height + body_width*body_width)}" iyz="0.0"
+    izz="${mass_body / 12.0 * (body_width*body_width + body_length*body_length)}"/>
     </inertial>
   </link>
@@ -80,9 +85,9 @@
     <inertial>
       <origin xyz="0 0 0" rpy="0 0 0"/>
-      <mass value="${mass}"/>
-      <inertia
-    ixx="${mass / 12.0*(block_length*block_length + block_height*block_height)}" ixy="0.0" ixz="0.0"
-    iyy="${mass / 12.0 * (block_height*block_height + block_width*block_width)}" iyz="0.0"
-    izz="${mass / 12.0 * (block_width*block_width + block_length*block_length)}"/>
+      <mass value="${mass_block}"/>
+      <inertia
+    ixx="${mass_block / 12.0*(block_length*block_length + block_height*block_height)}" ixy="0.0" ixz="0.0"
+    iyy="${mass_block / 12.0 * (block_height*block_height + block_width*block_width)}" iyz="0.0"
+    izz="${mass_block / 12.0 * (block_width*block_width + block_length*block_length)}"/>
     </inertial>
   </link>
@@ -103,9 +108,9 @@
     <inertial>
       <origin xyz="0 0 0" rpy="0 0 0"/>
-      <mass value="${mass}"/>
-      <inertia
-    ixx="${mass / 12.0*(block_length*block_length + block_height*block_height)}" ixy="0.0" ixz="0.0"
-    iyy="${mass / 12.0 * (block_height*block_height + block_width*block_width)}" iyz="0.0"
-    izz="${mass / 12.0 * (block_width*block_width + block_length*block_length)}"/>
+      <mass value="${mass_block}"/>
+      <inertia
+    ixx="${mass_block / 12.0*(block_length*block_length + block_height*block_height)}" ixy="0.0" ixz="0.0"
+    iyy="${mass_block / 12.0 * (block_height*block_height + block_width*block_width)}" iyz="0.0"
+    izz="${mass_block / 12.0 * (block_width*block_width + block_length*block_length)}"/>
     </inertial>
   </link>
@@ -126,9 +131,9 @@
     <inertial>
       <origin xyz="0 0 0" rpy="0 0 0"/>
-      <mass value="${mass}"/>
-      <inertia
-    ixx="${mass / 12.0*(block_length*block_length + block_height*block_height)}" ixy="0.0" ixz="0.0"
-    iyy="${mass / 12.0 * (block_height*block_height + block_width*block_width)}" iyz="0.0"
-    izz="${mass / 12.0 * (block_width*block_width + block_length*block_length)}"/>
+      <mass value="${mass_block}"/>
+      <inertia
+    ixx="${mass_block / 12.0*(block_length*block_length + block_height*block_height)}" ixy="0.0" ixz="0.0"
+    iyy="${mass_block / 12.0 * (block_height*block_height + block_width*block_width)}" iyz="0.0"
+    izz="${mass_block / 12.0 * (block_width*block_width + block_length*block_length)}"/>
     </inertial>
   </link>
@@ -149,9 +154,9 @@
     <inertial>
       <origin xyz="0 0 0" rpy="0 0 0"/>
-      <mass value="${mass}"/>
-      <inertia
-    ixx="${mass / 12.0*(block_length*block_length + block_height*block_height)}" ixy="0.0" ixz="0.0"
-    iyy="${mass / 12.0 * (block_height*block_height + block_width*block_width)}" iyz="0.0"
-    izz="${mass / 12.0 * (block_width*block_width + block_length*block_length)}"/>
+      <mass value="${mass_block}"/>
+      <inertia
+    ixx="${mass_block / 12.0*(block_length*block_length + block_height*block_height)}" ixy="0.0" ixz="0.0"
+    iyy="${mass_block / 12.0 * (block_height*block_height + block_width*block_width)}" iyz="0.0"
+    izz="${mass_block / 12.0 * (block_width*block_width + block_length*block_length)}"/>
     </inertial>
   </link>
@@ -185,5 +190,5 @@
     <origin xyz="${block_width/2} 0 0" rpy="0 0 -3.14"/>
     <axis xyz="0 0 1" />
-    <limit effort="30" velocity="1.0" lower="-1.7" upper="1.7"/>
+    <limit effort="300" velocity="1.0" lower="-1.7" upper="1.7"/>
   </joint>
     <joint name="hip_j2" type="revolute">
@@ -192,5 +197,5 @@
     <origin xyz="${block_width/2} 0 0" rpy="0 0 -3.14"/>
     <axis xyz="0 0 1" />
-    <limit effort="30" velocity="1.0" lower="-1.7" upper="1.7"/>
+    <limit effort="300" velocity="1.0" lower="-1.7" upper="1.7"/>
   </joint>
     <joint name="hip_j3" type="revolute">
@@ -199,5 +204,5 @@
     <origin xyz="${-block_width/2} 0 0" rpy="0 0 0"/>
     <axis xyz="0 0 1" />
-    <limit effort="30" velocity="1.0" lower="-1.7" upper="1.7"/>
+    <limit effort="300" velocity="1.0" lower="-1.7" upper="1.7"/>
   </joint>
     <joint name="hip_j4" type="revolute">
@@ -206,5 +211,5 @@
     <origin xyz="${-block_width/2} 0 0" rpy="0 0 0"/>
     <axis xyz="0 0 1" />
-    <limit effort="30" velocity="1.0" lower="-1.7" upper="1.7"/>
+    <limit effort="300" velocity="1.0" lower="-1.7" upper="1.7"/>
   </joint>
   <!-- Base Link -->
@@ -225,9 +230,9 @@
     <inertial>
       <origin xyz="${-hip_width/2} 0 0" rpy="0 0 0"/>
-      <mass value="${mass}"/>
-      <inertia
-	  ixx="${mass / 12.0 * (hip_length*hip_length + hip_height*hip_height)}" ixy="0.0" ixz="0.0"
-	  iyy="${mass / 12.0 * (hip_height*hip_height + hip_width*hip_width)}" iyz="0.0"
-	  izz="${mass / 12.0 * (hip_length*hip_length + hip_width*hip_width)}"/>
+      <mass value="${mass_hip}"/>
+      <inertia
+	  ixx="${mass_hip / 12.0 * (hip_length*hip_length + hip_height*hip_height)}" ixy="0.0" ixz="0.0"
+	  iyy="${mass_hip / 12.0 * (hip_height*hip_height + hip_width*hip_width)}" iyz="0.0"
+	  izz="${mass_hip / 12.0 * (hip_length*hip_length + hip_width*hip_width)}"/>
     </inertial>
   </link>
@@ -248,9 +253,9 @@
     <inertial>
       <origin xyz="${-hip_width/2} 0 0" rpy="0 0 0"/>
-      <mass value="${mass}"/>
-      <inertia
-    ixx="${mass / 12.0 * (hip_length*hip_length + hip_height*hip_height)}" ixy="0.0" ixz="0.0"
-    iyy="${mass / 12.0 * (hip_height*hip_height + hip_width*hip_width)}" iyz="0.0"
-    izz="${mass / 12.0 * (hip_length*hip_length + hip_width*hip_width)}"/>
+      <mass value="${mass_hip}"/>
+      <inertia
+    ixx="${mass_hip / 12.0 * (hip_length*hip_length + hip_height*hip_height)}" ixy="0.0" ixz="0.0"
+    iyy="${mass_hip / 12.0 * (hip_height*hip_height + hip_width*hip_width)}" iyz="0.0"
+    izz="${mass_hip / 12.0 * (hip_length*hip_length + hip_width*hip_width)}"/>
     </inertial>
   </link>
@@ -271,9 +276,9 @@
     <inertial>
       <origin xyz="${-hip_width/2} 0 0" rpy="0 0 0"/>
-      <mass value="${mass}"/>
-      <inertia
-    ixx="${mass / 12.0 * (hip_length*hip_length + hip_height*hip_height)}" ixy="0.0" ixz="0.0"
-    iyy="${mass / 12.0 * (hip_height*hip_height + hip_width*hip_width)}" iyz="0.0"
-    izz="${mass / 12.0 * (hip_length*hip_length + hip_width*hip_width)}"/>
+      <mass value="${mass_hip}"/>
+      <inertia
+    ixx="${mass_hip / 12.0 * (hip_length*hip_length + hip_height*hip_height)}" ixy="0.0" ixz="0.0"
+    iyy="${mass_hip / 12.0 * (hip_height*hip_height + hip_width*hip_width)}" iyz="0.0"
+    izz="${mass_hip / 12.0 * (hip_length*hip_length + hip_width*hip_width)}"/>
     </inertial>
   </link>
@@ -294,9 +299,9 @@
     <inertial>
       <origin xyz="${-hip_width/2} 0 0" rpy="0 0 0"/>
-      <mass value="${mass}"/>
-      <inertia
-    ixx="${mass / 12.0 * (hip_length*hip_length + hip_height*hip_height)}" ixy="0.0" ixz="0.0"
-    iyy="${mass / 12.0 * (hip_height*hip_height + hip_width*hip_width)}" iyz="0.0"
-    izz="${mass / 12.0 * (hip_length*hip_length + hip_width*hip_width)}"/>
+      <mass value="${mass_hip}"/>
+      <inertia
+    ixx="${mass_hip / 12.0 * (hip_length*hip_length + hip_height*hip_height)}" ixy="0.0" ixz="0.0"
+    iyy="${mass_hip / 12.0 * (hip_height*hip_height + hip_width*hip_width)}" iyz="0.0"
+    izz="${mass_hip / 12.0 * (hip_length*hip_length + hip_width*hip_width)}"/>
     </inertial>
   </link>
@@ -307,5 +312,5 @@
     <axis xyz="0 1 0"/>
     <dynamics damping="0.7"/>
-    <limit effort="30" velocity="1.0" lower="-1.7" upper="1.7"/>
+    <limit effort="300" velocity="1.0" lower="-1.7" upper="1.7"/>
   </joint>
   <joint name="knee_j2" type="revolute">
@@ -315,5 +320,5 @@
     <axis xyz="0 1 0"/>
     <dynamics damping="0.7"/>
-    <limit effort="30" velocity="1.0" lower="-1.7" upper="1.7"/>
+    <limit effort="300" velocity="1.0" lower="-1.7" upper="1.7"/>
   </joint>
   <joint name="knee_j3" type="revolute">
@@ -323,5 +328,5 @@
     <axis xyz="0 1 0"/>
     <dynamics damping="0.7"/>
-    <limit effort="30" velocity="1.0" lower="-1.7" upper="1.7"/>
+    <limit effort="300" velocity="1.0" lower="-1.7" upper="1.7"/>
   </joint>
   <joint name="knee_j4" type="revolute">
@@ -331,5 +336,5 @@
     <axis xyz="0 1 0"/>
     <dynamics damping="0.7"/>
-    <limit effort="30" velocity="1.0" lower="-1.7" upper="1.7"/>
+    <limit effort="300" velocity="1.0" lower="-1.7" upper="1.7"/>
   </joint>
   <!-- Middle Link -->
@@ -350,9 +355,9 @@
     <inertial>
       <origin xyz="0 0 ${leg_height/2}" rpy="0 0 0"/>
-      <mass value="${mass}"/>
-      <inertia
-	  ixx="${mass / 12.0 * (leg_length*leg_length + leg_height*leg_height)}" ixy="0.0" ixz="0.0"
-	  iyy="${mass / 12.0 * (leg_height*leg_height + leg_width*leg_width)}" iyz="0.0"
-	  izz="${mass / 12.0 * (leg_width*leg_width + leg_length*leg_length)}"/>
+      <mass value="${mass_leg}"/>
+      <inertia
+	  ixx="${mass_leg / 12.0 * (leg_length*leg_length + leg_height*leg_height)}" ixy="0.0" ixz="0.0"
+	  iyy="${mass_leg / 12.0 * (leg_height*leg_height + leg_width*leg_width)}" iyz="0.0"
+	  izz="${mass_leg / 12.0 * (leg_width*leg_width + leg_length*leg_length)}"/>
     </inertial>
   </link>
@@ -373,9 +378,9 @@
     <inertial>
       <origin xyz="0 0 ${leg_height/2}" rpy="0 0 0"/>
-      <mass value="${mass}"/>
-      <inertia
-    ixx="${mass / 12.0 * (leg_length*leg_length + leg_height*leg_height)}" ixy="0.0" ixz="0.0"
-    iyy="${mass / 12.0 * (leg_height*leg_height + leg_width*leg_width)}" iyz="0.0"
-    izz="${mass / 12.0 * (leg_width*leg_width + leg_length*leg_length)}"/>
+      <mass value="${mass_leg}"/>
+      <inertia
+    ixx="${mass_leg / 12.0 * (leg_length*leg_length + leg_height*leg_height)}" ixy="0.0" ixz="0.0"
+    iyy="${mass_leg / 12.0 * (leg_height*leg_height + leg_width*leg_width)}" iyz="0.0"
+    izz="${mass_leg / 12.0 * (leg_width*leg_width + leg_length*leg_length)}"/>
     </inertial>
   </link>
@@ -396,9 +401,9 @@
     <inertial>
       <origin xyz="0 0 ${leg_height/2}" rpy="0 0 0"/>
-      <mass value="${mass}"/>
-      <inertia
-    ixx="${mass / 12.0 * (leg_length*leg_length + leg_height*leg_height)}" ixy="0.0" ixz="0.0"
-    iyy="${mass / 12.0 * (leg_height*leg_height + leg_width*leg_width)}" iyz="0.0"
-    izz="${mass / 12.0 * (leg_width*leg_width + leg_length*leg_length)}"/>
+      <mass value="${mass_leg}"/>
+      <inertia
+    ixx="${mass_leg / 12.0 * (leg_length*leg_length + leg_height*leg_height)}" ixy="0.0" ixz="0.0"
+    iyy="${mass_leg / 12.0 * (leg_height*leg_height + leg_width*leg_width)}" iyz="0.0"
+    izz="${mass_leg / 12.0 * (leg_width*leg_width + leg_length*leg_length)}"/>
     </inertial>
   </link>
@@ -419,9 +424,9 @@
     <inertial>
       <origin xyz="0 0 ${leg_height/2}" rpy="0 0 0"/>
-      <mass value="${mass}"/>
-      <inertia
-    ixx="${mass / 12.0 * (leg_length*leg_length + leg_height*leg_height)}" ixy="0.0" ixz="0.0"
-    iyy="${mass / 12.0 * (leg_height*leg_height + leg_width*leg_width)}" iyz="0.0"
-    izz="${mass / 12.0 * (leg_width*leg_width + leg_length*leg_length)}"/>
+      <mass value="${mass_leg}"/>
+      <inertia
+    ixx="${mass_leg / 12.0 * (leg_length*leg_length + leg_height*leg_height)}" ixy="0.0" ixz="0.0"
+    iyy="${mass_leg / 12.0 * (leg_height*leg_height + leg_width*leg_width)}" iyz="0.0"
+    izz="${mass_leg / 12.0 * (leg_width*leg_width + leg_length*leg_length)}"/>
     </inertial>
   </link>
@@ -432,5 +437,5 @@
     <axis xyz="0 1 0"/>
     <dynamics damping="0.7"/>
-    <limit effort="30" velocity="1.0" lower="-3" upper="3"/>
+    <limit effort="300" velocity="1.0" lower="-1.7" upper="1.7"/>
   </joint>
   <joint name="ankle_j2" type="revolute">
@@ -440,5 +445,5 @@
     <axis xyz="0 1 0"/>
     <dynamics damping="0.7"/>
-    <limit effort="30" velocity="1.0" lower="-1.7" upper="1.7"/>
+    <limit effort="300" velocity="1.0" lower="-1.7" upper="1.7"/>
   </joint>
   <joint name="ankle_j3" type="revolute">
@@ -448,5 +453,5 @@
     <axis xyz="0 1 0"/>
     <dynamics damping="0.7"/>
-    <limit effort="30" velocity="1.0" lower="-1.7" upper="1.7"/>
+    <limit effort="300" velocity="1.0" lower="-1.7" upper="1.7"/>
   </joint>
   <joint name="ankle_j4" type="revolute">
@@ -456,5 +461,5 @@
     <axis xyz="0 1 0"/>
     <dynamics damping="0.7"/>
-    <limit effort="30" velocity="1.0" lower="-1.7" upper="1.7"/>
+    <limit effort="300" velocity="1.0" lower="-1.7" upper="1.7"/>
   </joint>
   <!-- Top Link -->
@@ -475,9 +480,9 @@
     <inertial>
       <origin xyz="0 0 ${foot_height/2}" rpy="0 0 0"/>
-      <mass value="${mass}"/>
-      <inertia
-	  ixx="${mass / 12.0 * (foot_length*foot_length + foot_height*foot_height)}" ixy="0.0" ixz="0.0"
-	  iyy="${mass / 12.0 * (foot_width*foot_width + foot_height*foot_height)}" iyz="0.0"
-	  izz="${mass / 12.0 * (foot_width*foot_width + foot_length*foot_length)}"/>
+      <mass value="${mass_foot}"/>
+      <inertia
+	  ixx="${mass_foot / 12.0 * (foot_length*foot_length + foot_height*foot_height)}" ixy="0.0" ixz="0.0"
+	  iyy="${mass_foot / 12.0 * (foot_width*foot_width + foot_height*foot_height)}" iyz="0.0"
+	  izz="${mass_foot / 12.0 * (foot_width*foot_width + foot_length*foot_length)}"/>
     </inertial>
   </link>
@@ -498,9 +503,9 @@
     <inertial>
       <origin xyz="0 0 ${foot_height/2}" rpy="0 0 0"/>
-      <mass value="${mass}"/>
-      <inertia
-    ixx="${mass / 12.0 * (foot_length*foot_length + foot_height*foot_height)}" ixy="0.0" ixz="0.0"
-    iyy="${mass / 12.0 * (foot_width*foot_width + foot_height*foot_height)}" iyz="0.0"
-    izz="${mass / 12.0 * (foot_width*foot_width + foot_length*foot_length)}"/>
+      <mass value="${mass_foot}"/>
+      <inertia
+    ixx="${mass_foot / 12.0 * (foot_length*foot_length + foot_height*foot_height)}" ixy="0.0" ixz="0.0"
+    iyy="${mass_foot / 12.0 * (foot_width*foot_width + foot_height*foot_height)}" iyz="0.0"
+    izz="${mass_foot / 12.0 * (foot_width*foot_width + foot_length*foot_length)}"/>
     </inertial>
   </link>
@@ -521,9 +526,9 @@
     <inertial>
       <origin xyz="0 0 ${foot_height/2}" rpy="0 0 0"/>
-      <mass value="${mass}"/>
-      <inertia
-    ixx="${mass / 12.0 * (foot_length*foot_length + foot_height*foot_height)}" ixy="0.0" ixz="0.0"
-    iyy="${mass / 12.0 * (foot_width*foot_width + foot_height*foot_height)}" iyz="0.0"
-    izz="${mass / 12.0 * (foot_width*foot_width + foot_length*foot_length)}"/>
+      <mass value="${mass_foot}"/>
+      <inertia
+    ixx="${mass_foot / 12.0 * (foot_length*foot_length + foot_height*foot_height)}" ixy="0.0" ixz="0.0"
+    iyy="${mass_foot / 12.0 * (foot_width*foot_width + foot_height*foot_height)}" iyz="0.0"
+    izz="${mass_foot / 12.0 * (foot_width*foot_width + foot_length*foot_length)}"/>
     </inertial>
   </link>
@@ -544,74 +549,10 @@
     <inertial>
       <origin xyz="0 0 ${foot_height/2}" rpy="0 0 0"/>
-      <mass value="${mass}"/>
-      <inertia
-    ixx="${mass / 12.0 * (foot_length*foot_length + foot_height*foot_height)}" ixy="0.0" ixz="0.0"
-    iyy="${mass / 12.0 * (foot_width*foot_width + foot_height*foot_height)}" iyz="0.0"
-    izz="${mass / 12.0 * (foot_width*foot_width + foot_length*foot_length)}"/>
-    </inertial>
-  </link>
-  <joint name="hokuyo_joint" type="fixed">
-    <axis xyz="0 1 0" />
-    <origin xyz="0 0 ${height3 - axel_offset/2}" rpy="0 0 0"/>
-    <parent link="foot1"/>
-    <child link="hokuyo_link"/>
-  </joint>
-  <!-- Hokuyo Laser -->
-  <link name="hokuyo_link">
-    <collision>
-      <origin xyz="0 0 0" rpy="0 0 0"/>
-      <geometry>
-	<box size="0.001 0.001 0.001"/>
-      </geometry>
-    </collision>
-    <visual>
-      <origin xyz="0 0 0" rpy="0 0 0"/>
-      <geometry>
-        <mesh filename="package://rrbot_description/meshes/hokuyo.dae"/>
-      </geometry>
-    </visual>
-    <inertial>
-      <mass value="1e-5" />
-      <origin xyz="0 0 0" rpy="0 0 0"/>
-      <inertia ixx="1e-6" ixy="0" ixz="0" iyy="1e-6" iyz="0" izz="1e-6" />
-    </inertial>
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